File: kicadfiles/summerday/summerday.kicad_pcb (KiCad board)
At the start: 2 copper layers, 278.4 x 93.1 mm, 106 parts, among them J1 USB_C_Receptacle_USB2.0_14P, SW1 SW_DPST_x2, SW2 SW_DPST_x2, U1 XC6206PxxxMR, U2 STM32F072CBTx, U3 SRV05-4

Commit message: updated pcb artworks
Parts:
- R1: value R6_5.1k -> 5.1k
- R2: value R7_5.1k -> 5.1k
- moved C8 317.6 mm to (200.1, 109.4), turned to -5 degrees
- moved C4 311.0 mm to (206.8, 130.9), turned to 180 degrees
- moved C3 304.8 mm to (210.1, 134.2), turned to -90 degrees
- moved C5 303.7 mm to (214.4, 134.2), turned to -90 degrees
- moved C2 303.3 mm to (210.0, 121.8), turned to 90 degrees
- moved R1 299.7 mm to (211.9, 107.7), turned to -90 degrees
- moved F1 298.4 mm to (217.5, 109.2), turned to -90 degrees
- moved C7 297.9 mm to (221.0, 117.7)
- moved C9 296.8 mm to (220.2, 101.5), turned to 5 degrees
- moved R2 296.5 mm to (215.0, 107.7), turned to -90 degrees
- moved C1 295.0 mm to (219.2, 125.3)
- moved C6 295.0 mm to (220.0, 112.6)
- moved U2 293.9 mm to (213.0, 128.0), turned to 90 degrees
- moved R3 290.8 mm to (220.2, 100.3), turned to 5 degrees
- moved U3 287.5 mm to (213.4, 111.8), turned to 90 degrees
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- renumbered SW2 to BOOT, SW1 to RST
Routing:
- net ROW1: track 0.00 -> 165.7 mm, vias 0 -> 6
- net ROW0: track 0.00 -> 111.0 mm, vias 0 -> 1
- net ROW2: track 0.00 -> 110.6 mm
- net COL3: track 0.00 -> 90.9 mm
- net ROW3: track 0.00 -> 88.4 mm
- net COL2: track 0.00 -> 86.6 mm
- net COL4: track 0.00 -> 75.0 mm
- net COL5: track 0.00 -> 66.5 mm
- net +3V3: track 0.00 -> 62.3 mm
- net COL1: track 0.00 -> 43.7 mm
- net COL0: track 0.00 -> 40.1 mm
- net BOOT-1: track 0.00 -> 38.5 mm, vias 0 -> 2
- net RST-1: track 0.00 -> 36.1 mm
- net DP: track 0.00 -> 22.3 mm
- net DN: track 0.00 -> 22.2 mm
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