File: kicadfiles/summerday/summerday.kicad_pcb (KiCad board)
At the start: 2 copper layers, 278.4 x 93.1 mm, 106 parts, among them J1 USB_C_Receptacle_USB2.0_14P, U1 XC6206PxxxMR, U2 STM32F072CBTx, U3 SRV05-4

Commit message: Almost Finished pcb artworks
Parts:
- moved R4 7.17 mm to (227.9, 130.2), turned to -85 degrees
- moved C1 0.40 mm to (219.3, 124.9)
- renumbered RST to SW1, BOOT to SW2
Connections:
- U2 pad 14: unconnected-(U2-PA4-Pad14) -> ROW2
- U2 pad 15: unconnected-(U2-PA5-Pad15) -> ROW3
- U2 pad 17: unconnected-(U2-PA7-Pad17) -> COL6
- U2 pad 18: unconnected-(U2-PB0-Pad18) -> COL7
- U2 pad 19: unconnected-(U2-PB1-Pad19) -> COL8
- U2 pad 20: unconnected-(U2-PB2-Pad20) -> COL9
- U2 pad 21: unconnected-(U2-PB10-Pad21) -> COL10
- U2 pad 22: unconnected-(U2-PB11-Pad22) -> COL11
- U2 pad 27: unconnected-(U2-PB14-Pad27) -> ROW0
- U2 pad 28: unconnected-(U2-PB15-Pad28) -> ROW1
- U2 pad 37: unconnected-(U2-PA14-Pad37) -> COL0
- U2 pad 38: unconnected-(U2-PA15-Pad38) -> COL1
- U2 pad 39: unconnected-(U2-PB3-Pad39) -> COL2
- U2 pad 40: unconnected-(U2-PB4-Pad40) -> COL3
- U2 pad 41: unconnected-(U2-PB5-Pad41) -> COL4
- U2 pad 42: unconnected-(U2-PB6-Pad42) -> COL5
Routing:
- net ROW0: track 111.0 -> 338.6 mm, vias 1 -> 15
- net ROW2: track 110.6 -> 325.5 mm, vias 0 -> 13
- net ROW3: track 88.4 -> 289.3 mm, vias 0 -> 9
- net COL10: track 0.00 -> 170.1 mm, vias 0 -> 2
- net COL9: track 0.00 -> 167.1 mm, vias 0 -> 2
- net COL11: track 0.00 -> 163.3 mm, vias 0 -> 2
- net COL8: track 0.00 -> 145.0 mm, vias 0 -> 2
- net COL0: track 40.1 -> 166.2 mm, vias 0 -> 2
- net COL7: track 0.00 -> 118.7 mm, vias 0 -> 2
- net ROW1: track 165.7 -> 281.4 mm, vias 6 -> 12
- net COL1: track 43.7 -> 148.8 mm, vias 0 -> 2
- net COL6: track 0.00 -> 100.7 mm
- net COL2: track 86.6 -> 171.2 mm, vias 0 -> 2
- net COL3: track 90.9 -> 159.2 mm, vias 0 -> 2
- net COL4: track 75.0 -> 124.3 mm, vias 0 -> 2
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- added copper zone on B.Cu, net GND
- added copper zone on F.Cu, net GND
Other:
- board text added: "Boot"
- board text added: "Reset"
